File: tinynfc/kicad/tinynfc.kicad_sch (KiCad schematic)
At the start: 15 parts, among them Q1 DMP21D0UFB4, U1 NT3H2111W0FHKH, U2 ATtiny816-MNR

Commit message: Shrink TinyNFC to 28 mm postage stamp, not card size
Drop the outline from 40 mm to 28 mm with a 23 mm / 6-turn spiral, switch
to a 9×9 FUET-9018 piezo so the island fits, hide footprint silk refs that
were landing on copper, and refresh BOM/design costs for the smaller board.

Co-authored-by: Jason Hall <imjasonh@users.noreply.github.com>
Parts:
- PZ1: value PKLCS1212E4001-R1 -> FUET-9018; footprint Buzzer_Beeper:Buzzer_Murata_PKLCS1212E -> Buzzer_Beeper:Buzzer_Murata_PKMCS0909E
- TP1, TP2, TP3: footprint TestPoint:TestPoint_Pad_D1.5mm -> TestPoint:TestPoint_Pad_D1.0mm
Changed lines of the file:
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@@
     (instances
       (project "tinynfc"
-        (path "/51170c99-d51a-4c54-a128-94b6372bedf6"
+        (path "/4ef393b9-bae8-4c6e-a5a4-b22b3982fd5f"
           (reference "U1")
           (unit 1)
@@
     (instances
       (project "tinynfc"
-        (path "/51170c99-d51a-4c54-a128-94b6372bedf6"
+        (path "/4ef393b9-bae8-4c6e-a5a4-b22b3982fd5f"
           (reference "L1")
           (unit 1)
@@
     (instances
       (project "tinynfc"
-        (path "/51170c99-d51a-4c54-a128-94b6372bedf6"
+        (path "/4ef393b9-bae8-4c6e-a5a4-b22b3982fd5f"
           (reference "C1")
           (unit 1)
@@
     (instances
       (project "tinynfc"
-        (path "/51170c99-d51a-4c54-a128-94b6372bedf6"
+        (path "/4ef393b9-bae8-4c6e-a5a4-b22b3982fd5f"
           (reference "C2")
           (unit 1)
@@
     (instances
       (project "tinynfc"
-        (path "/51170c99-d51a-4c54-a128-94b6372bedf6"
+        (path "/4ef393b9-bae8-4c6e-a5a4-b22b3982fd5f"
           (reference "Q1")
           (unit 1)
@@
     (instances
       (project "tinynfc"
-        (path "/51170c99-d51a-4c54-a128-94b6372bedf6"
+        (path "/4ef393b9-bae8-4c6e-a5a4-b22b3982fd5f"
           (reference "R1")
           (unit 1)
@@
     (instances
       (project "tinynfc"
-        (path "/51170c99-d51a-4c54-a128-94b6372bedf6"
+        (path "/4ef393b9-bae8-4c6e-a5a4-b22b3982fd5f"
           (reference "R2")
           (unit 1)
@@
     (instances
       (project "tinynfc"
-        (path "/51170c99-d51a-4c54-a128-94b6372bedf6"
+        (path "/4ef393b9-bae8-4c6e-a5a4-b22b3982fd5f"
           (reference "C3")
           (unit 1)
@@
     (instances
       (project "tinynfc"
-        (path "/51170c99-d51a-4c54-a128-94b6372bedf6"
+        (path "/4ef393b9-bae8-4c6e-a5a4-b22b3982fd5f"
           (reference "U2")
           (unit 1)
@@
     (instances
       (project "tinynfc"
-        (path "/51170c99-d51a-4c54-a128-94b6372bedf6"
+        (path "/4ef393b9-bae8-4c6e-a5a4-b22b3982fd5f"
           (reference "R3")
           (unit 1)
@@
     (property "Reference" "PZ1" (at 241.3 71.12 0)
       (effects (font (size 1.27 1.27))))
-    (property "Value" "PKLCS1212E4001-R1" (at 241.3 81.28 0)
-      (effects (font (size 1.27 1.27))))
-    (property "Footprint" "Buzzer_Beeper:Buzzer_Murata_PKLCS1212E" (at 241.3 76.2 0)
+    (property "Value" "FUET-9018" (at 241.3 81.28 0)
+      (effects (font (size 1.27 1.27))))
+    (property "Footprint" "Buzzer_Beeper:Buzzer_Murata_PKMCS0909E" (at 241.3 76.2 0)
       (effects (font (size 1.27 1.27)) hide))
     (property "Datasheet" "" (at 241.3 76.2 0)
       (effects (font (size 1.27 1.27)) hide))
-    (pin "1")
-    (pin "2")
-    (instances
-      (project "tinynfc"
-        (path "/51170c99-d51a-4c54-a128-94b6372bedf6"
+    (property "Description" "9x9 passive piezo; PKMCS0909 land pattern" (at 241.3 76.2 0)
+      (effects (font (size 1.27 1.27)) hide))
+    (pin "1")
+    (pin "2")
+    (instances
+      (project "tinynfc"
+        (path "/4ef393b9-bae8-4c6e-a5a4-b22b3982fd5f"
           (reference "PZ1")
           (unit 1)
@@
     (property "Value" "GND" (at 101.6 106.67999999999999 0)
       (effects (font (size 1.27 1.27))))
-    (property "Footprint" "TestPoint:TestPoint_Pad_D1.5mm" (at 101.6 101.6 0)
+    (property "Footprint" "TestPoint:TestPoint_Pad_D1.0mm" (at 101.6 101.6 0)
       (effects (font (size 1.27 1.27)) hide))
     (property "Datasheet" "" (at 101.6 101.6 0)
@@
     (instances
       (project "tinynfc"
-        (path "/51170c99-d51a-4c54-a128-94b6372bedf6"
+        (path "/4ef393b9-bae8-4c6e-a5a4-b22b3982fd5f"
           (reference "TP1")
           (unit 1)
@@
     (property "Value" "VCC" (at 111.76 106.67999999999999 0)
       (effects (font (size 1.27 1.27))))
-    (property "Footprint" "TestPoint:TestPoint_Pad_D1.5mm" (at 111.76 101.6 0)
+    (property "Footprint" "TestPoint:TestPoint_Pad_D1.0mm" (at 111.76 101.6 0)
       (effects (font (size 1.27 1.27)) hide))
     (property "Datasheet" "" (at 111.76 101.6 0)
@@
     (instances
       (project "tinynfc"
-        (path "/51170c99-d51a-4c54-a128-94b6372bedf6"
+        (path "/4ef393b9-bae8-4c6e-a5a4-b22b3982fd5f"
           (reference "TP2")
           (unit 1)
@@
     (property "Value" "UPDI" (at 121.92 106.67999999999999 0)
       (effects (font (size 1.27 1.27))))
-    (property "Footprint" "TestPoint:TestPoint_Pad_D1.5mm" (at 121.92 101.6 0)
+    (property "Footprint" "TestPoint:TestPoint_Pad_D1.0mm" (at 121.92 101.6 0)
       (effects (font (size 1.27 1.27)) hide))
     (property "Datasheet" "" (at 121.92 101.6 0)
@@
     (instances
       (project "tinynfc"
-        (path "/51170c99-d51a-4c54-a128-94b6372bedf6"
+        (path "/4ef393b9-bae8-4c6e-a5a4-b22b3982fd5f"
           (reference "TP3")
           (unit 1)
@@
     (instances
       (project "tinynfc"
-        (path "/51170c99-d51a-4c54-a128-94b6372bedf6"
+        (path "/4ef393b9-bae8-4c6e-a5a4-b22b3982fd5f"
           (reference "D1")
           (unit 1)
@@
     (instances
       (project "tinynfc"
-        (path "/51170c99-d51a-4c54-a128-94b6372bedf6"
+        (path "/4ef393b9-bae8-4c6e-a5a4-b22b3982fd5f"
           (reference "#FLG01")
           (unit 1)
@@
     (instances
       (project "tinynfc"
-        (path "/51170c99-d51a-4c54-a128-94b6372bedf6"
+        (path "/4ef393b9-bae8-4c6e-a5a4-b22b3982fd5f"
           (reference "#PWR01")
           (unit 1)

Commit message: Make TinyNFC board and antenna circular
Switch the Edge.Cuts outline to Ø 28 mm and replace the square spiral with
a Ø 24 mm Archimedean spiral so the coil matches phone NFC geometry better.
Update design, BOM, and README for the round postage-stamp disc.

Co-authored-by: Jason Hall <imjasonh@users.noreply.github.com>
Parts:
- L1: footprint tinynfc:PCB_Antenna_RectSpiral -> tinynfc:PCB_Antenna_RoundSpiral
Changed lines of the file:
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@@
     (instances
       (project "tinynfc"
-        (path "/47a1e2c1-95d2-46a0-bbe7-ea5318d08ef7"
+        (path "/19c61324-5beb-4473-9e79-3e404d081f1c"
           (reference "U1")
           (unit 1)
@@
     (property "Value" "2.75uH" (at 33.02 58.42 0)
       (effects (font (size 1.27 1.27))))
-    (property "Footprint" "tinynfc:PCB_Antenna_RectSpiral" (at 33.02 53.34 0)
+    (property "Footprint" "tinynfc:PCB_Antenna_RoundSpiral" (at 33.02 53.34 0)
       (effects (font (size 1.27 1.27)) hide))
     (property "Datasheet" "" (at 33.02 53.34 0)
@@
     (instances
       (project "tinynfc"
-        (path "/47a1e2c1-95d2-46a0-bbe7-ea5318d08ef7"
+        (path "/19c61324-5beb-4473-9e79-3e404d081f1c"
           (reference "L1")
           (unit 1)
@@
     (instances
       (project "tinynfc"
-        (path "/47a1e2c1-95d2-46a0-bbe7-ea5318d08ef7"
+        (path "/19c61324-5beb-4473-9e79-3e404d081f1c"
           (reference "C1")
           (unit 1)
@@
     (instances
       (project "tinynfc"
-        (path "/47a1e2c1-95d2-46a0-bbe7-ea5318d08ef7"
+        (path "/19c61324-5beb-4473-9e79-3e404d081f1c"
           (reference "C2")
           (unit 1)
@@
     (instances
       (project "tinynfc"
-        (path "/47a1e2c1-95d2-46a0-bbe7-ea5318d08ef7"
+        (path "/19c61324-5beb-4473-9e79-3e404d081f1c"
           (reference "Q1")
           (unit 1)
@@
     (instances
       (project "tinynfc"
-        (path "/47a1e2c1-95d2-46a0-bbe7-ea5318d08ef7"
+        (path "/19c61324-5beb-4473-9e79-3e404d081f1c"
           (reference "R1")
           (unit 1)
@@
     (instances
       (project "tinynfc"
-        (path "/47a1e2c1-95d2-46a0-bbe7-ea5318d08ef7"
+        (path "/19c61324-5beb-4473-9e79-3e404d081f1c"
           (reference "R2")
           (unit 1)
@@
     (instances
       (project "tinynfc"
-        (path "/47a1e2c1-95d2-46a0-bbe7-ea5318d08ef7"
+        (path "/19c61324-5beb-4473-9e79-3e404d081f1c"
           (reference "C3")
           (unit 1)
@@
     (instances
       (project "tinynfc"
-        (path "/47a1e2c1-95d2-46a0-bbe7-ea5318d08ef7"
+        (path "/19c61324-5beb-4473-9e79-3e404d081f1c"
           (reference "U2")
           (unit 1)
@@
     (instances
       (project "tinynfc"
-        (path "/47a1e2c1-95d2-46a0-bbe7-ea5318d08ef7"
+        (path "/19c61324-5beb-4473-9e79-3e404d081f1c"
           (reference "R3")
           (unit 1)
@@
     (instances
       (project "tinynfc"
-        (path "/47a1e2c1-95d2-46a0-bbe7-ea5318d08ef7"
+        (path "/19c61324-5beb-4473-9e79-3e404d081f1c"
           (reference "PZ1")
           (unit 1)
@@
     (instances
       (project "tinynfc"
-        (path "/47a1e2c1-95d2-46a0-bbe7-ea5318d08ef7"
+        (path "/19c61324-5beb-4473-9e79-3e404d081f1c"
           (reference "TP1")
           (unit 1)
@@
     (instances
       (project "tinynfc"
-        (path "/47a1e2c1-95d2-46a0-bbe7-ea5318d08ef7"
+        (path "/19c61324-5beb-4473-9e79-3e404d081f1c"
           (reference "TP2")
           (unit 1)
@@
     (instances
       (project "tinynfc"
-        (path "/47a1e2c1-95d2-46a0-bbe7-ea5318d08ef7"
+        (path "/19c61324-5beb-4473-9e79-3e404d081f1c"
           (reference "TP3")
           (unit 1)
@@
     (instances
       (project "tinynfc"
-        (path "/47a1e2c1-95d2-46a0-bbe7-ea5318d08ef7"
+        (path "/19c61324-5beb-4473-9e79-3e404d081f1c"
           (reference "D1")
           (unit 1)
@@
     (instances
       (project "tinynfc"
-        (path "/47a1e2c1-95d2-46a0-bbe7-ea5318d08ef7"
+        (path "/19c61324-5beb-4473-9e79-3e404d081f1c"
           (reference "#FLG01")
           (unit 1)
@@
     (instances
       (project "tinynfc"
-        (path "/47a1e2c1-95d2-46a0-bbe7-ea5318d08ef7"
+        (path "/19c61324-5beb-4473-9e79-3e404d081f1c"
           (reference "#PWR01")
           (unit 1)
