File: nfc-eink/mcu.kicad_sch (KiCad schematic)
At the start: 9 parts, among them J2 SWD, J3 UART, U5 STM32G071CBT6

Commit message: Fix first-article failures in the NFC e-ink design
The NTAG session masks were swapped, so pass-through never enabled
and the mailbox polled I2C_LOCKED. Hold EPD_PWR_EN and NRST at
reset, drop the push-pull reset cap, and use a low-profile tank so
a phone can sit on the coil.

Co-authored-by: Jason Hall <imjasonh@users.noreply.github.com>
Parts:
- J3: value UART -> UART DNP; now not fitted
- R7, R8: value 2.2k -> 4.7k; MPN RC0402FR-072K2L -> RC0402FR-074K7L
Changed lines of the file:
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@@
     (instances
       (project "nfc-eink"
-        (path "/f9a18703-a337-49ac-b86a-4c7a7cdf298f/7b3dc7ef-68d7-4134-ab75-23a33da7c27e"
+        (path "/9ad5f43f-f38f-4382-a467-b5b9de5a6ce4/ef93d21c-acef-4a91-81e0-c175b6688d93"
           (reference "U5") (unit 1)))))
   (symbol (lib_id "Device:C") (at 230 40 0) (unit 1)
@@
     (instances
       (project "nfc-eink"
-        (path "/f9a18703-a337-49ac-b86a-4c7a7cdf298f/7b3dc7ef-68d7-4134-ab75-23a33da7c27e"
+        (path "/9ad5f43f-f38f-4382-a467-b5b9de5a6ce4/ef93d21c-acef-4a91-81e0-c175b6688d93"
           (reference "C9") (unit 1)))))
   (symbol (lib_id "Device:C") (at 255 40 0) (unit 1)
@@
     (instances
       (project "nfc-eink"
-        (path "/f9a18703-a337-49ac-b86a-4c7a7cdf298f/7b3dc7ef-68d7-4134-ab75-23a33da7c27e"
+        (path "/9ad5f43f-f38f-4382-a467-b5b9de5a6ce4/ef93d21c-acef-4a91-81e0-c175b6688d93"
           (reference "C10") (unit 1)))))
   (symbol (lib_id "Device:C") (at 280 40 0) (unit 1)
@@
     (instances
       (project "nfc-eink"
-        (path "/f9a18703-a337-49ac-b86a-4c7a7cdf298f/7b3dc7ef-68d7-4134-ab75-23a33da7c27e"
+        (path "/9ad5f43f-f38f-4382-a467-b5b9de5a6ce4/ef93d21c-acef-4a91-81e0-c175b6688d93"
           (reference "C11") (unit 1)))))
   (symbol (lib_id "Device:R") (at 230 70 0) (unit 1)
@@
     (property "Reference" "R7" (at 230 62.38 0)
       (effects (font (size 1.27 1.27))))
-    (property "Value" "2.2k" (at 230 77.62 0)
+    (property "Value" "4.7k" (at 230 77.62 0)
       (effects (font (size 1.27 1.27))))
     (property "Footprint" "Resistor_SMD:R_0402_1005Metric" (at 230 70 0)
@@
     (property "Datasheet" "~" (at 230 70 0)
       (effects (font (size 1.27 1.27)) hide))
-    (property "MPN" "RC0402FR-072K2L" (at 230 70 0) (effects (font (size 1.27 1.27)) hide))
+    (property "MPN" "RC0402FR-074K7L" (at 230 70 0) (effects (font (size 1.27 1.27)) hide))
     (pin "1")
     (pin "2")
     (instances
       (project "nfc-eink"
-        (path "/f9a18703-a337-49ac-b86a-4c7a7cdf298f/7b3dc7ef-68d7-4134-ab75-23a33da7c27e"
+        (path "/9ad5f43f-f38f-4382-a467-b5b9de5a6ce4/ef93d21c-acef-4a91-81e0-c175b6688d93"
           (reference "R7") (unit 1)))))
   (symbol (lib_id "Device:R") (at 255 70 0) (unit 1)
@@
     (property "Reference" "R8" (at 255 62.38 0)
       (effects (font (size 1.27 1.27))))
-    (property "Value" "2.2k" (at 255 77.62 0)
+    (property "Value" "4.7k" (at 255 77.62 0)
       (effects (font (size 1.27 1.27))))
     (property "Footprint" "Resistor_SMD:R_0402_1005Metric" (at 255 70 0)
@@
     (property "Datasheet" "~" (at 255 70 0)
       (effects (font (size 1.27 1.27)) hide))
-    (property "MPN" "RC0402FR-072K2L" (at 255 70 0) (effects (font (size 1.27 1.27)) hide))
+    (property "MPN" "RC0402FR-074K7L" (at 255 70 0) (effects (font (size 1.27 1.27)) hide))
     (pin "1")
     (pin "2")
     (instances
       (project "nfc-eink"
-        (path "/f9a18703-a337-49ac-b86a-4c7a7cdf298f/7b3dc7ef-68d7-4134-ab75-23a33da7c27e"
+        (path "/9ad5f43f-f38f-4382-a467-b5b9de5a6ce4/ef93d21c-acef-4a91-81e0-c175b6688d93"
           (reference "R8") (unit 1)))))
   (symbol (lib_id "Device:R") (at 280 70 0) (unit 1)
@@
     (instances
       (project "nfc-eink"
-        (path "/f9a18703-a337-49ac-b86a-4c7a7cdf298f/7b3dc7ef-68d7-4134-ab75-23a33da7c27e"
+        (path "/9ad5f43f-f38f-4382-a467-b5b9de5a6ce4/ef93d21c-acef-4a91-81e0-c175b6688d93"
           (reference "R9") (unit 1)))))
   (symbol (lib_id "Connector:Conn_01x05_Pin") (at 50 220 0) (unit 1)
@@
     (instances
       (project "nfc-eink"
-        (path "/f9a18703-a337-49ac-b86a-4c7a7cdf298f/7b3dc7ef-68d7-4134-ab75-23a33da7c27e"
+        (path "/9ad5f43f-f38f-4382-a467-b5b9de5a6ce4/ef93d21c-acef-4a91-81e0-c175b6688d93"
           (reference "J2") (unit 1)))))
   (symbol (lib_id "Connector:Conn_01x03_Pin") (at 120 220 0) (unit 1)
-    (in_bom yes) (on_board yes) (dnp no)
+    (in_bom yes) (on_board yes) (dnp yes)
     (property "Reference" "J3" (at 120 212.38 0)
       (effects (font (size 1.27 1.27))))
-    (property "Value" "UART" (at 120 227.62 0)
+    (property "Value" "UART DNP" (at 120 227.62 0)
       (effects (font (size 1.27 1.27))))
     (property "Footprint" "Connector_PinHeader_2.54mm:PinHeader_1x03_P2.54mm_Vertical" (at 120 220 0)
@@
     (instances
       (project "nfc-eink"
-        (path "/f9a18703-a337-49ac-b86a-4c7a7cdf298f/7b3dc7ef-68d7-4134-ab75-23a33da7c27e"
+        (path "/9ad5f43f-f38f-4382-a467-b5b9de5a6ce4/ef93d21c-acef-4a91-81e0-c175b6688d93"
           (reference "J3") (unit 1)))))
   (symbol (lib_id "power:+3V3") (at 360 40 0) (unit 1)
@@
     (instances
       (project "nfc-eink"
-        (path "/f9a18703-a337-49ac-b86a-4c7a7cdf298f/7b3dc7ef-68d7-4134-ab75-23a33da7c27e"
+        (path "/9ad5f43f-f38f-4382-a467-b5b9de5a6ce4/ef93d21c-acef-4a91-81e0-c175b6688d93"
           (reference "#PWR001P") (unit 1)))))
   (symbol (lib_id "power:GND") (at 360 60 0) (unit 1)
@@
     (instances
       (project "nfc-eink"
-        (path "/f9a18703-a337-49ac-b86a-4c7a7cdf298f/7b3dc7ef-68d7-4134-ab75-23a33da7c27e"
+        (path "/9ad5f43f-f38f-4382-a467-b5b9de5a6ce4/ef93d21c-acef-4a91-81e0-c175b6688d93"
           (reference "#PWR002G") (unit 1)))))
   (sheet_instances
-    (path "/f9a18703-a337-49ac-b86a-4c7a7cdf298f/7b3dc7ef-68d7-4134-ab75-23a33da7c27e" (page "4"))
+    (path "/9ad5f43f-f38f-4382-a467-b5b9de5a6ce4/ef93d21c-acef-4a91-81e0-c175b6688d93" (page "4"))
   )
 )
