File: nfc-eink/nfc-eink.kicad_pcb (KiCad board)
At the start: 4 copper layers, 91 x 77 mm, 44 parts, among them J1 FH12-24S-0.5SH, J2 SWD, J3 UART, Q1 2N7002, U1 NT3H2211W0FTTJ, U2 TPS61023DRLR, U3 TPS22917DBVR, U4 TCM809SENB713, U5 STM32G071CBT6

Commit message: Fix first-article failures in the NFC e-ink design
The NTAG session masks were swapped, so pass-through never enabled
and the mailbox polled I2C_LOCKED. Hold EPD_PWR_EN and NRST at
reset, drop the push-pull reset cap, and use a low-profile tank so
a phone can sit on the coil.

Co-authored-by: Jason Hall <imjasonh@users.noreply.github.com>
Parts:
- removed C8: 100nF, C_0402_1005Metric
- added R11: 100k, R_0402_1005Metric, F.Cu at (68.0, 32.0)
- added R12: 100k, R_0402_1005Metric, F.Cu at (68.0, 28.0)
- C2: value 470uF -> 470uF POSCAP; footprint CP_Radial_D8.0mm_P3.50mm -> CP_EIA-7343-20_Kemet-V
- J3: value UART -> UART DNP
- R7, R8: value 2.2k -> 4.7k
- moved C2 2.00 mm to (18.0, 20.0)
Routing:
- net NFC_LB: track 0.00 -> 24.2 mm
- net NFC_LA: track 685.3 -> 661.1 mm
- net EPD_PWR_EN: track 17.4 -> 25.6 mm
- net GND: track 24.3 -> 26.1 mm, vias 27 -> 29
- net VSTORE: track 5.40 -> 6.30 mm, vias 6 -> 7
Other:
- board text added: "J2 bring-up only. J3 DNP. FPC contacts toward board."
