File: inkbot-magsafe/kicad/inkbot-magsafe.kicad_sch (KiCad schematic)
At the start: 77 parts, among them J1 GDEY0397T81P panel FPC, J2 Protected battery + NTC, J3 WR222230 coil + bonded NTC, Q1 Si1308EDL-T1-GE3, Q2 2N7002BK,215, U1 MDBT50Q-512K, U2 BQ51013C, U3 BQ25186DLHR, U4 TPS7A2030PDBVR, U5 TPS7A0230PDBVR, Y1 FC-135 32.768kHz 12.5pF

Commit message: inkbot-magsafe: close follow-up DFM gaps
Co-authored-by: Jason Hall <imjasonh@users.noreply.github.com>
Parts:
- BT1: value LP242030 100mAh 2C protected -> LP242030 100mAh protected HR
- C30, C36: value 1uF 50V -> 1uF 50V X5R
- C31, C32, C33, C34, C35, C37: value 4.7uF 25V -> 4.7uF 50V X7R; footprint Capacitor_SMD:C_0805_2012Metric -> Capacitor_SMD:C_1206_3216Metric
- RT2: value 10k 3435K coil NTC -> 103JT-025 10k 3435K film NTC
Changed lines of the file:
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@@
     (property "Reference" "RT2" (at 165.10 60.96 0)
       (effects (font (size 1.27 1.27))))
-    (property "Value" "10k 3435K coil NTC" (at 165.10 68.58 0)
+    (property "Value" "103JT-025 10k 3435K film NTC" (at 165.10 68.58 0)
       (effects (font (size 1.0 1.0))))
     (property "Footprint" "" (at 165.10 69.85 0)
@@
     (property "Reference" "BT1" (at 275.59 86.36 0)
       (effects (font (size 1.27 1.27))))
-    (property "Value" "LP242030 100mAh 2C protected" (at 275.59 93.98 0)
+    (property "Value" "LP242030 100mAh protected HR" (at 275.59 93.98 0)
       (effects (font (size 1.0 1.0))))
     (property "Footprint" "" (at 275.59 95.25 0)
@@
     (property "Reference" "C30" (at 340.36 176.53 0)
       (effects (font (size 1.27 1.27))))
-    (property "Value" "1uF 50V" (at 340.36 184.15 0)
+    (property "Value" "1uF 50V X5R" (at 340.36 184.15 0)
       (effects (font (size 1.0 1.0))))
     (property "Footprint" "Capacitor_SMD:C_0603_1608Metric" (at 340.36 185.42 0)
@@
     (property "Reference" "C31" (at 350.52 176.53 0)
       (effects (font (size 1.27 1.27))))
-    (property "Value" "4.7uF 25V" (at 350.52 184.15 0)
-      (effects (font (size 1.0 1.0))))
-    (property "Footprint" "Capacitor_SMD:C_0805_2012Metric" (at 350.52 185.42 0)
+    (property "Value" "4.7uF 50V X7R" (at 350.52 184.15 0)
+      (effects (font (size 1.0 1.0))))
+    (property "Footprint" "Capacitor_SMD:C_1206_3216Metric" (at 350.52 185.42 0)
       (effects (font (size 1.27 1.27)) hide))
     (property "LCSC" "" (at 350.52 186.69 0)
@@
     (property "Reference" "C32" (at 359.41 176.53 0)
       (effects (font (size 1.27 1.27))))
-    (property "Value" "4.7uF 25V" (at 359.41 184.15 0)
-      (effects (font (size 1.0 1.0))))
-    (property "Footprint" "Capacitor_SMD:C_0805_2012Metric" (at 359.41 185.42 0)
+    (property "Value" "4.7uF 50V X7R" (at 359.41 184.15 0)
+      (effects (font (size 1.0 1.0))))
+    (property "Footprint" "Capacitor_SMD:C_1206_3216Metric" (at 359.41 185.42 0)
       (effects (font (size 1.27 1.27)) hide))
     (property "LCSC" "" (at 359.41 186.69 0)
@@
     (property "Reference" "C33" (at 369.57 176.53 0)
       (effects (font (size 1.27 1.27))))
-    (property "Value" "4.7uF 25V" (at 369.57 184.15 0)
-      (effects (font (size 1.0 1.0))))
-    (property "Footprint" "Capacitor_SMD:C_0805_2012Metric" (at 369.57 185.42 0)
+    (property "Value" "4.7uF 50V X7R" (at 369.57 184.15 0)
+      (effects (font (size 1.0 1.0))))
+    (property "Footprint" "Capacitor_SMD:C_1206_3216Metric" (at 369.57 185.42 0)
       (effects (font (size 1.27 1.27)) hide))
     (property "LCSC" "" (at 369.57 186.69 0)
@@
     (property "Reference" "C34" (at 379.73 176.53 0)
       (effects (font (size 1.27 1.27))))
-    (property "Value" "4.7uF 25V" (at 379.73 184.15 0)
-      (effects (font (size 1.0 1.0))))
-    (property "Footprint" "Capacitor_SMD:C_0805_2012Metric" (at 379.73 185.42 0)
+    (property "Value" "4.7uF 50V X7R" (at 379.73 184.15 0)
+      (effects (font (size 1.0 1.0))))
+    (property "Footprint" "Capacitor_SMD:C_1206_3216Metric" (at 379.73 185.42 0)
       (effects (font (size 1.27 1.27)) hide))
     (property "LCSC" "" (at 379.73 186.69 0)
@@
     (property "Reference" "C35" (at 389.89 176.53 0)
       (effects (font (size 1.27 1.27))))
-    (property "Value" "4.7uF 25V" (at 389.89 184.15 0)
-      (effects (font (size 1.0 1.0))))
-    (property "Footprint" "Capacitor_SMD:C_0805_2012Metric" (at 389.89 185.42 0)
+    (property "Value" "4.7uF 50V X7R" (at 389.89 184.15 0)
+      (effects (font (size 1.0 1.0))))
+    (property "Footprint" "Capacitor_SMD:C_1206_3216Metric" (at 389.89 185.42 0)
       (effects (font (size 1.27 1.27)) hide))
     (property "LCSC" "" (at 389.89 186.69 0)
@@
     (property "Reference" "C36" (at 400.05 176.53 0)
       (effects (font (size 1.27 1.27))))
-    (property "Value" "1uF 50V" (at 400.05 184.15 0)
+    (property "Value" "1uF 50V X5R" (at 400.05 184.15 0)
       (effects (font (size 1.0 1.0))))
     (property "Footprint" "Capacitor_SMD:C_0603_1608Metric" (at 400.05 185.42 0)
@@
     (property "Reference" "C37" (at 374.65 130.81 0)
       (effects (font (size 1.27 1.27))))
-    (property "Value" "4.7uF 25V" (at 374.65 138.43 0)
-      (effects (font (size 1.0 1.0))))
-    (property "Footprint" "Capacitor_SMD:C_0805_2012Metric" (at 374.65 139.70 0)
+    (property "Value" "4.7uF 50V X7R" (at 374.65 138.43 0)
+      (effects (font (size 1.0 1.0))))
+    (property "Footprint" "Capacitor_SMD:C_1206_3216Metric" (at 374.65 139.70 0)
       (effects (font (size 1.27 1.27)) hide))
     (property "LCSC" "" (at 374.65 140.97 0)

Commit message: inkbot-magsafe: qualify panel and sensing parts
Co-authored-by: Jason Hall <imjasonh@users.noreply.github.com>
Parts:
- C31, C32, C33, C34, C35, C37: value 4.7uF 50V X7R -> 4.7uF 35V X7R; footprint Capacitor_SMD:C_1206_3216Metric -> Capacitor_SMD:C_0805_2012Metric
Changed lines of the file:
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@@
     (property "Reference" "C31" (at 350.52 176.53 0)
       (effects (font (size 1.27 1.27))))
-    (property "Value" "4.7uF 50V X7R" (at 350.52 184.15 0)
+    (property "Value" "4.7uF 35V X7R" (at 350.52 184.15 0)
       (effects (font (size 1.0 1.0))))
-    (property "Footprint" "Capacitor_SMD:C_1206_3216Metric" (at 350.52 185.42 0)
+    (property "Footprint" "Capacitor_SMD:C_0805_2012Metric" (at 350.52 185.42 0)
       (effects (font (size 1.27 1.27)) hide))
     (property "LCSC" "" (at 350.52 186.69 0)
@@
     (property "Reference" "C32" (at 359.41 176.53 0)
       (effects (font (size 1.27 1.27))))
-    (property "Value" "4.7uF 50V X7R" (at 359.41 184.15 0)
+    (property "Value" "4.7uF 35V X7R" (at 359.41 184.15 0)
       (effects (font (size 1.0 1.0))))
-    (property "Footprint" "Capacitor_SMD:C_1206_3216Metric" (at 359.41 185.42 0)
+    (property "Footprint" "Capacitor_SMD:C_0805_2012Metric" (at 359.41 185.42 0)
       (effects (font (size 1.27 1.27)) hide))
     (property "LCSC" "" (at 359.41 186.69 0)
@@
     (property "Reference" "C33" (at 369.57 176.53 0)
       (effects (font (size 1.27 1.27))))
-    (property "Value" "4.7uF 50V X7R" (at 369.57 184.15 0)
+    (property "Value" "4.7uF 35V X7R" (at 369.57 184.15 0)
       (effects (font (size 1.0 1.0))))
-    (property "Footprint" "Capacitor_SMD:C_1206_3216Metric" (at 369.57 185.42 0)
+    (property "Footprint" "Capacitor_SMD:C_0805_2012Metric" (at 369.57 185.42 0)
       (effects (font (size 1.27 1.27)) hide))
     (property "LCSC" "" (at 369.57 186.69 0)
@@
     (property "Reference" "C34" (at 379.73 176.53 0)
       (effects (font (size 1.27 1.27))))
-    (property "Value" "4.7uF 50V X7R" (at 379.73 184.15 0)
+    (property "Value" "4.7uF 35V X7R" (at 379.73 184.15 0)
       (effects (font (size 1.0 1.0))))
-    (property "Footprint" "Capacitor_SMD:C_1206_3216Metric" (at 379.73 185.42 0)
+    (property "Footprint" "Capacitor_SMD:C_0805_2012Metric" (at 379.73 185.42 0)
       (effects (font (size 1.27 1.27)) hide))
     (property "LCSC" "" (at 379.73 186.69 0)
@@
     (property "Reference" "C35" (at 389.89 176.53 0)
       (effects (font (size 1.27 1.27))))
-    (property "Value" "4.7uF 50V X7R" (at 389.89 184.15 0)
+    (property "Value" "4.7uF 35V X7R" (at 389.89 184.15 0)
       (effects (font (size 1.0 1.0))))
-    (property "Footprint" "Capacitor_SMD:C_1206_3216Metric" (at 389.89 185.42 0)
+    (property "Footprint" "Capacitor_SMD:C_0805_2012Metric" (at 389.89 185.42 0)
       (effects (font (size 1.27 1.27)) hide))
     (property "LCSC" "" (at 389.89 186.69 0)
@@
     (property "Reference" "C37" (at 374.65 130.81 0)
       (effects (font (size 1.27 1.27))))
-    (property "Value" "4.7uF 50V X7R" (at 374.65 138.43 0)
+    (property "Value" "4.7uF 35V X7R" (at 374.65 138.43 0)
       (effects (font (size 1.0 1.0))))
-    (property "Footprint" "Capacitor_SMD:C_1206_3216Metric" (at 374.65 139.70 0)
+    (property "Footprint" "Capacitor_SMD:C_0805_2012Metric" (at 374.65 139.70 0)
       (effects (font (size 1.27 1.27)) hide))
     (property "LCSC" "" (at 374.65 140.97 0)

Commit message: inkbot-magsafe: add measurable panel temperature
Co-authored-by: Jason Hall <imjasonh@users.noreply.github.com>
Parts:
- removed D2: MBR0530, Diode_SMD:D_SOD-123, symbol Device:D
- added R13: 10k 1%, Resistor_SMD:R_0603_1608Metric, symbol Device:R
- added RT3: NCP18XH103F03RB 10k 3380K, Capacitor_SMD:C_0603_1608Metric, symbol Device:Thermistor_NTC
- added TP2: SWDCLK, TestPoint:TestPoint_Pad_D1.0mm, symbol Connector:TestPoint
- D2: renamed from TP2; value SWDCLK -> MBR0530; footprint TestPoint:TestPoint_Pad_D1.0mm -> Diode_SMD:D_SOD-123; symbol Connector:TestPoint -> Device:D
Connections:
- net EP: now also D2.1 (K), U1.32 (VBUS), RT3.2
- net PANEL_PUMP: now also D2.2 (A)
- net SWDCLK: now also TP2.1; no longer D2.1
- net PANEL_TEMP_SENSE: now reaches U1.13 (P0.28)
- net PANEL_TEMP_SENSE: now also R13.2, RT3.1
- net PANEL_TEMP_EXCITE: now reaches U1.16 (P0.27)
- net PANEL_TEMP_EXCITE: now also R13.1
- no-connect marks 45 -> 42
Changed lines of the file:
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@@
+    )
+  )
+  (symbol (lib_id "Device:R") (at 234.95 175.26 0)
+    (property "Reference" "R13" (at 234.95 171.45 0)
+      (effects (font (size 1.27 1.27))))
+    (property "Value" "10k 1%" (at 234.95 179.07 0)
+      (effects (font (size 1.0 1.0))))
+    (property "Footprint" "Resistor_SMD:R_0603_1608Metric" (at 234.95 180.34 0)
+      (effects (font (size 1.27 1.27)) hide))
+    (property "LCSC" "" (at 234.95 181.61 0)
+      (effects (font (size 1.27 1.27)) hide))
+    (instances
+      (project "inkbot-magsafe"
+        (path "/876e0bc8-f839-529d-8fb7-fca7b9334b7c" (reference "R13") (unit 1))
+      )
+    )
+  )
+  (symbol (lib_id "Device:Thermistor_NTC") (at 245.11 175.26 0)
+    (property "Reference" "RT3" (at 245.11 171.45 0)
+      (effects (font (size 1.27 1.27))))
+    (property "Value" "NCP18XH103F03RB 10k 3380K" (at 245.11 179.07 0)
+      (effects (font (size 1.0 1.0))))
+    (property "Footprint" "Capacitor_SMD:C_0603_1608Metric" (at 245.11 180.34 0)
+      (effects (font (size 1.27 1.27)) hide))
+    (property "LCSC" "" (at 245.11 181.61 0)
+      (effects (font (size 1.27 1.27)) hide))
+    (instances
+      (project "inkbot-magsafe"
+        (path "/876e0bc8-f839-529d-8fb7-fca7b9334b7c" (reference "RT3") (unit 1))
+      )
     )
   )
@@
     (stroke (width 0) (type default))
   )
+  (wire (pts (xy 134.62 212.09) (xy 124.46 212.09))
+    (stroke (width 0) (type default))
+  )
   (wire (pts (xy 134.62 217.17) (xy 124.46 217.17))
     (stroke (width 0) (type default))
   )
+  (wire (pts (xy 175.26 255.27) (xy 185.42 255.27))
+    (stroke (width 0) (type default))
+  )
   (wire (pts (xy 175.26 199.39) (xy 185.42 199.39))
     (stroke (width 0) (type default))
@@
     (stroke (width 0) (type default))
   )
+  (wire (pts (xy 157.48 189.23) (xy 157.48 196.85))
+    (stroke (width 0) (type default))
+  )
   (wire (pts (xy 175.26 219.71) (xy 185.42 219.71))
     (stroke (width 0) (type default))
@@
     (stroke (width 0) (type default))
   )
+  (wire (pts (xy 234.95 171.45) (xy 234.95 168.91))
+    (stroke (width 0) (type default))
+  )
+  (wire (pts (xy 234.95 179.07) (xy 234.95 181.61))
+    (stroke (width 0) (type default))
+  )
+  (wire (pts (xy 245.11 171.45) (xy 245.11 168.91))
+    (stroke (width 0) (type default))
+  )
+  (wire (pts (xy 245.11 179.07) (xy 245.11 181.61))
+    (stroke (width 0) (type default))
+  )
   (wire (pts (xy 229.87 171.45) (xy 229.87 168.91))
     (stroke (width 0) (type default))
@@
     (effects (font (size 1.27 1.27)) (justify left))
   )
+  (label "PANEL_TEMP_SENSE" (at 124.46 212.09 0)
+    (effects (font (size 1.27 1.27)) (justify left))
+  )
   (label "PANEL_BUSY" (at 124.46 217.17 0)
     (effects (font (size 1.27 1.27)) (justify left))
   )
+  (label "PANEL_TEMP_EXCITE" (at 185.42 255.27 0)
+    (effects (font (size 1.27 1.27)) (justify left))
+  )
   (label "XL1" (at 185.42 199.39 0)
     (effects (font (size 1.27 1.27)) (justify left))
@@
     (effects (font (size 1.27 1.27)) (justify left))
   )
+  (label "GND" (at 157.48 196.85 0)
+    (effects (font (size 1.27 1.27)) (justify left))
+  )
   (label "PANEL_MOSI" (at 185.42 219.71 0)
     (effects (font (size 1.27 1.27)) (justify left))
@@
     (effects (font (size 1.27 1.27)) (justify left))
   )
+  (label "PANEL_TEMP_EXCITE" (at 234.95 168.91 0)
+    (effects (font (size 1.27 1.27)) (justify left))
+  )
+  (label "PANEL_TEMP_SENSE" (at 234.95 181.61 0)
+    (effects (font (size 1.27 1.27)) (justify left))
+  )
+  (label "PANEL_TEMP_SENSE" (at 245.11 168.91 0)
+    (effects (font (size 1.27 1.27)) (justify left))
+  )
+  (label "GND" (at 245.11 181.61 0)
+    (effects (font (size 1.27 1.27)) (justify left))
+  )
   (label "SYS" (at 229.87 168.91 0)
     (effects (font (size 1.27 1.27)) (justify left))
@@
   (no_connect (at 104.14 67.31)
   )
-  (no_connect (at 134.62 212.09)
-  )
   (no_connect (at 154.94 280.67)
   )
-  (no_connect (at 175.26 255.27)
-  )
   (no_connect (at 175.26 252.73)
   )
@@
   (no_connect (at 160.02 191.77)
   )
-  (no_connect (at 157.48 189.23)
-  )
   (no_connect (at 154.94 280.67)

Commit message: inkbot-magsafe: harden state and frame persistence
Co-authored-by: Jason Hall <imjasonh@users.noreply.github.com>
Parts:
- U1: value MDBT50Q-512K -> MDBT50Q-1MV2; symbol RF_Module:MDBT50Q-512K -> RF_Module:MDBT50Q-1MV2
Other:
- note added: "inkbot-magsafe EVT schematic BQ51013C Qi 1.3 receiver + BQ25186 protected-cell charger, Raytac MDBT50Q-1MV2 on a nanopower 3.0 V rail, and the GDEY0397T81P SSD1677 boost circuit. Qi resonance and FOD values require EVT tuning."
- note removed: "inkbot-magsafe EVT schematic BQ51013C Qi 1.3 receiver + BQ25186 protected-cell charger, Raytac MDBT50Q-512K on a nanopower 3.0 V rail, and the GDEY0397T81P SSD1677 boost circuit. Qi resonance and FOD values require EVT tuning."
Changed lines of the file:
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@@
     )
   )
-  (symbol (lib_id "RF_Module:MDBT50Q-512K") (at 154.94 234.95 0)
+  (symbol (lib_id "RF_Module:MDBT50Q-1MV2") (at 154.94 234.95 0)
     (property "Reference" "U1" (at 154.94 231.14 0)
       (effects (font (size 1.27 1.27))))
-    (property "Value" "MDBT50Q-512K" (at 154.94 238.76 0)
+    (property "Value" "MDBT50Q-1MV2" (at 154.94 238.76 0)
       (effects (font (size 1.0 1.0))))
     (property "Footprint" "RF_Module:Raytac_MDBT50Q" (at 154.94 240.03 0)
@@
     (stroke (width 0) (type default))
   )
-  (wire (pts (xy 134.62 275.59) (xy 124.46 275.59))
+  (wire (pts (xy 134.62 260.35) (xy 124.46 260.35))
     (stroke (width 0) (type default))
   )
@@
     (effects (font (size 1.27 1.27)) (justify left))
   )
-  (label "QI_EN2" (at 124.46 275.59 0)
+  (label "QI_EN2" (at 124.46 260.35 0)
     (effects (font (size 1.27 1.27)) (justify left))
   )
@@
   (no_connect (at 175.26 262.89)
   )
+  (no_connect (at 134.62 262.89)
+  )
+  (no_connect (at 160.02 189.23)
+  )
+  (no_connect (at 154.94 280.67)
+  )
+  (no_connect (at 134.62 234.95)
+  )
+  (no_connect (at 134.62 237.49)
+  )
+  (no_connect (at 175.26 217.17)
+  )
+  (no_connect (at 175.26 214.63)
+  )
+  (no_connect (at 175.26 222.25)
+  )
+  (no_connect (at 134.62 265.43)
+  )
+  (no_connect (at 175.26 234.95)
+  )
+  (no_connect (at 175.26 240.03)
+  )
+  (no_connect (at 175.26 245.11)
+  )
+  (no_connect (at 175.26 242.57)
+  )
+  (no_connect (at 175.26 260.35)
+  )
+  (no_connect (at 175.26 247.65)
+  )
+  (no_connect (at 175.26 250.19)
+  )
+  (no_connect (at 134.62 267.97)
+  )
+  (no_connect (at 134.62 245.11)
+  )
+  (no_connect (at 134.62 224.79)
+  )
+  (no_connect (at 134.62 227.33)
+  )
+  (no_connect (at 154.94 280.67)
+  )
   (no_connect (at 134.62 250.19)
   )
-  (no_connect (at 160.02 191.77)
-  )
-  (no_connect (at 154.94 280.67)
-  )
-  (no_connect (at 134.62 234.95)
-  )
-  (no_connect (at 134.62 237.49)
-  )
-  (no_connect (at 175.26 217.17)
-  )
-  (no_connect (at 175.26 214.63)
-  )
-  (no_connect (at 175.26 222.25)
-  )
-  (no_connect (at 137.16 252.73)
-  )
-  (no_connect (at 172.72 234.95)
-  )
-  (no_connect (at 175.26 240.03)
-  )
-  (no_connect (at 172.72 245.11)
-  )
-  (no_connect (at 175.26 242.57)
-  )
-  (no_connect (at 175.26 260.35)
-  )
-  (no_connect (at 175.26 247.65)
-  )
-  (no_connect (at 172.72 250.19)
+  (no_connect (at 134.62 255.27)
+  )
+  (no_connect (at 134.62 257.81)
+  )
+  (no_connect (at 134.62 252.73)
+  )
+  (no_connect (at 134.62 270.51)
   )
   (no_connect (at 134.62 247.65)
   )
-  (no_connect (at 134.62 260.35)
-  )
-  (no_connect (at 134.62 224.79)
-  )
-  (no_connect (at 134.62 227.33)
-  )
-  (no_connect (at 154.94 280.67)
-  )
-  (no_connect (at 134.62 265.43)
-  )
-  (no_connect (at 134.62 270.51)
+  (no_connect (at 134.62 242.57)
   )
   (no_connect (at 134.62 273.05)
   )
-  (no_connect (at 172.72 196.85)
-  )
-  (no_connect (at 134.62 267.97)
-  )
-  (no_connect (at 172.72 194.31)
-  )
-  (no_connect (at 134.62 257.81)
-  )
-  (no_connect (at 134.62 262.89)
-  )
-  (no_connect (at 134.62 245.11)
+  (no_connect (at 134.62 275.59)
   )
   (no_connect (at 74.93 149.86)
@@
   (no_connect (at 340.36 252.73)
   )
-  (text "inkbot-magsafe EVT schematic\nBQ51013C Qi 1.3 receiver + BQ25186 protected-cell charger,\nRaytac MDBT50Q-512K on a nanopower 3.0 V rail, and the GDEY0397T81P\nSSD1677 boost circuit. Qi resonance and FOD values require EVT tuning." (at 15.24 15.24 0)
+  (text "inkbot-magsafe EVT schematic\nBQ51013C Qi 1.3 receiver + BQ25186 protected-cell charger,\nRaytac MDBT50Q-1MV2 on a nanopower 3.0 V rail, and the GDEY0397T81P\nSSD1677 boost circuit. Qi resonance and FOD values require EVT tuning." (at 15.24 15.24 0)
     (effects (font (size 2.54 2.54)) (justify left))
   )

Commit message: inkbot-magsafe: remove redundant power flags
Co-authored-by: Jason Hall <imjasonh@users.noreply.github.com>
Changed lines of the file:
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@@
-    )
-  )
-  (symbol (lib_id "power:PWR_FLAG") (at 224.79 39.37 0)
-    (property "Reference" "#FLG001" (at 224.79 41.91 0)
-      (effects (font (size 1.27 1.27)) hide))
-    (property "Value" "PWR_FLAG" (at 224.79 43.18 0)
-      (effects (font (size 0.8 0.8))))
-    (property "Footprint" "" (at 224.79 39.37 0)
-      (effects (font (size 1.27 1.27)) hide))
-    (instances
-      (project "inkbot-magsafe"
-        (path "/876e0bc8-f839-529d-8fb7-fca7b9334b7c" (reference "#FLG001") (unit 1))
-      )
-    )
-  )
-  (symbol (lib_id "power:PWR_FLAG") (at 234.95 39.37 0)
-    (property "Reference" "#FLG002" (at 234.95 41.91 0)
-      (effects (font (size 1.27 1.27)) hide))
-    (property "Value" "PWR_FLAG" (at 234.95 43.18 0)
-      (effects (font (size 0.8 0.8))))
-    (property "Footprint" "" (at 234.95 39.37 0)
-      (effects (font (size 1.27 1.27)) hide))
-    (instances
-      (project "inkbot-magsafe"
-        (path "/876e0bc8-f839-529d-8fb7-fca7b9334b7c" (reference "#FLG002") (unit 1))
-      )
-    )
-  )
-  (symbol (lib_id "power:PWR_FLAG") (at 294.64 124.46 0)
-    (property "Reference" "#FLG003" (at 294.64 127.00 0)
-      (effects (font (size 1.27 1.27)) hide))
-    (property "Value" "PWR_FLAG" (at 294.64 128.27 0)
-      (effects (font (size 0.8 0.8))))
-    (property "Footprint" "" (at 294.64 124.46 0)
-      (effects (font (size 1.27 1.27)) hide))
-    (instances
-      (project "inkbot-magsafe"
-        (path "/876e0bc8-f839-529d-8fb7-fca7b9334b7c" (reference "#FLG003") (unit 1))
-      )
-    )
-  )
-  (symbol (lib_id "power:PWR_FLAG") (at 69.85 185.42 0)
-    (property "Reference" "#FLG004" (at 69.85 187.96 0)
-      (effects (font (size 1.27 1.27)) hide))
-    (property "Value" "PWR_FLAG" (at 69.85 189.23 0)
-      (effects (font (size 0.8 0.8))))
-    (property "Footprint" "" (at 69.85 185.42 0)
-      (effects (font (size 1.27 1.27)) hide))
-    (instances
-      (project "inkbot-magsafe"
-        (path "/876e0bc8-f839-529d-8fb7-fca7b9334b7c" (reference "#FLG004") (unit 1))
-      )
     )
   )
@@
     (effects (font (size 1.27 1.27)) (justify left))
   )
-  (label "SYS" (at 224.79 39.37 0)
-    (effects (font (size 1.27 1.27)) (justify left))
-  )
-  (label "BAT" (at 234.95 39.37 0)
-    (effects (font (size 1.27 1.27)) (justify left))
-  )
-  (label "PANEL_3V0" (at 294.64 124.46 0)
-    (effects (font (size 1.27 1.27)) (justify left))
-  )
-  (label "MCU_3V0" (at 69.85 185.42 0)
-    (effects (font (size 1.27 1.27)) (justify left))
-  )
